File: helix_minimal.kicad_pcb (KiCad board)
At the start: 2 copper layers, 50 x 50 mm, 20 parts, among them J1 USB-C, J4 sd card, J5 SWD, J6 pico hdmi, U1 STM32C071FBP6, U2 AP2112K-3.3, U3 WIZ850io

Commit message: autoroute
Parts:
- moved H2 24.8 mm to (90.0, 125.0)
- moved H1 23.5 mm to (90.0, 85.0)
- moved H4 23.4 mm to (130.0, 125.0)
- moved J4 22.8 mm to (131.4, 111.0)
- moved C1 22.8 mm to (102.1, 91.9)
- moved C3 22.8 mm to (97.1, 111.5)
- moved J1 22.8 mm to (102.2, 83.7)
- moved J6 22.8 mm to (91.3, 91.3)
- moved R2 22.8 mm to (102.1, 97.0)
- moved U1 22.8 mm to (102.1, 111.1)
- moved U2 22.8 mm to (102.1, 101.9)
- moved C2 22.8 mm to (94.5, 111.5)
- moved J5 22.8 mm to (97.7, 123.7)
- moved R1 22.8 mm to (102.1, 94.4)
- moved R5 22.8 mm to (122.5, 114.1)
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